Commit message: feat: Absorb unitree-go2-ros2 and add scalable model

File: install/go2_description/share/go2_description/xacro/const.xacro (robot description, xacro)
@@ -1,26 +1,32 @@
 <?xml version="1.0"?>
 <robot xmlns:xacro="http://www.ros.org/wiki/xacro">
+    <!-- Constants for robot dimensions -->
     <xacro:property name="PI" value="3.1415926535897931"/>
     <xacro:property name="stick_mass" value="0.00001"/>
-    <xacro:property name="trunk_width" value="0.0735"/>
-    <xacro:property name="trunk_length" value="0.08762"/>
-    <xacro:property name="trunk_height" value="0.0714"/>
-    <xacro:property name="hip_radius" value="0.022"/>
-    <xacro:property name="hip_length" value="0.03"/>
-    <xacro:property name="thigh_shoulder_radius" value="0.021"/>
+    <!-- simplified collision value -->
+    <xacro:property name="trunk_width" value="0.0935"/>
+    <xacro:property name="trunk_length" value="0.3762"/>
+    <xacro:property name="trunk_height" value="0.114"/>
+    <xacro:property name="hip_radius" value="0.046"/>
+    <xacro:property name="hip_length" value="0.04"/>
+    <xacro:property name="thigh_shoulder_radius" value="0.041"/>
     <xacro:property name="thigh_shoulder_length" value="0.032"/>
     <xacro:property name="thigh_width" value="0.0245"/>
-    <xacro:property name="thigh_height" value="0.024"/>
+    <xacro:property name="thigh_height" value="0.034"/>
     <xacro:property name="calf_width" value="0.016"/>
     <xacro:property name="calf_height" value="0.016"/>
-    <xacro:property name="foot_radius" value="0.015"/>
+    <xacro:property name="foot_radius" value="0.01"/>
     <xacro:property name="stick_radius" value="0.01"/>
     <xacro:property name="stick_length" value="0.2"/>
-    <xacro:property name="thigh_offset" value="0.049313"/>
-    <xacro:property name="thigh_length" value="0.059896"/>
-    <xacro:property name="calf_length" value="0.04"/>
-    <xacro:property name="leg_offset_x" value="0.075"/>
-    <xacro:property name="leg_offset_y" value="0.022462"/>
-    <xacro:property name="hip_offset" value="-0.015"/>
+    <!-- kinematic value -->
+    <xacro:property name="thigh_offset" value="0.0955"/>
+    <xacro:property name="thigh_length" value="0.1"/>
+    <xacro:property name="calf_length" value="0.133"/>
+    <!-- leg offset from trunk center value -->
+    <xacro:property name="leg_offset_x" value="0.1934"/>
+    <xacro:property name="leg_offset_y" value="0.0465"/>
+    <!-- <xacro:property name="trunk_offset_z" value="0.01675"/> -->
+    <xacro:property name="hip_offset" value="-0.03"/>
+    <!-- offset of link locations (left front) -->
     <xacro:property name="hip_offset_x" value="0.1934"/>
     <xacro:property name="hip_offset_y" value="0.0465"/>
@@ -32,4 +38,5 @@
     <xacro:property name="calf_offset_y" value="0.0"/>
     <xacro:property name="calf_offset_z" value="-0.213"/>
+    <!-- joint limits -->
     <xacro:property name="damping" value="0.01"/>
     <xacro:property name="friction" value="0.2"/>
@@ -46,8 +53,10 @@
     <xacro:property name="calf_velocity_max" value="20.06"/>
     <xacro:property name="calf_torque_max" value="80.0"/>
-    <xacro:property name="trunk_mass" value="1.521"/>
-    <xacro:property name="trunk_com_x" value="0.0"/>
-    <xacro:property name="trunk_com_y" value="0.0"/>
-    <xacro:property name="trunk_com_z" value="0.03"/>
+    <!-- dynamics inertial value -->
+    <!-- trunk -->
+    <xacro:property name="trunk_mass" value="1.921"/>
+    <xacro:property name="trunk_com_x" value="0.11112"/>
+    <xacro:property name="trunk_com_y" value="0.00"/>
+    <xacro:property name="trunk_com_z" value="-0.005366"/>
     <xacro:property name="trunk_ixx" value="0.02448"/>
     <xacro:property name="trunk_ixy" value="0.00012166"/>
@@ -56,8 +65,9 @@
     <xacro:property name="trunk_iyz" value="-3.12E-05"/>
     <xacro:property name="trunk_izz" value="0.107"/>
+    <!-- hip (left front) -->
     <xacro:property name="hip_mass" value="0.378"/>
-    <xacro:property name="hip_com_x" value="0.0"/>
-    <xacro:property name="hip_com_y" value="0.0"/>
-    <xacro:property name="hip_com_z" value="0.02"/>
+    <xacro:property name="hip_com_x" value="-0.0054"/>
+    <xacro:property name="hip_com_y" value="0.00194"/>
+    <xacro:property name="hip_com_z" value="-0.000105"/>
     <xacro:property name="hip_ixx" value="0.00048"/>
     <xacro:property name="hip_ixy" value="-3.01E-06"/>
@@ -66,8 +76,9 @@
     <xacro:property name="hip_iyz" value="-1.42E-06"/>
     <xacro:property name="hip_izz" value="0.000596"/>
+    <!-- thigh -->
     <xacro:property name="thigh_mass" value="0.152"/>
-    <xacro:property name="thigh_com_x" value="0.0"/>
-    <xacro:property name="thigh_com_y" value="-0.02"/>
-    <xacro:property name="thigh_com_z" value="-0.03"/>
+    <xacro:property name="thigh_com_x" value="-0.00374"/>
+    <xacro:property name="thigh_com_y" value="-0.0323"/>
+    <xacro:property name="thigh_com_z" value="-0.0327"/>
     <xacro:property name="thigh_ixx" value="0.00584"/>
     <xacro:property name="thigh_ixy" value="8.72E-05"/>
@@ -76,8 +87,9 @@
     <xacro:property name="thigh_iyz" value="0.000808"/>
     <xacro:property name="thigh_izz" value="0.00103"/>
-    <xacro:property name="calf_mass" value="0.025"/>
-    <xacro:property name="calf_com_x" value="-0.02"/>
-    <xacro:property name="calf_com_y" value="-0.02"/>
-    <xacro:property name="calf_com_z" value="-0.03"/>
+    <!-- calf -->
+    <xacro:property name="calf_mass" value="0.154"/>
+    <xacro:property name="calf_com_x" value="-0.0374"/>
+    <xacro:property name="calf_com_y" value="-0.0323"/>
+    <xacro:property name="calf_com_z" value="-0.0115"/>
     <xacro:property name="calf_ixx" value="0.00108"/>
     <xacro:property name="calf_ixy" value="3.4E-07"/>
@@ -86,4 +98,5 @@
     <xacro:property name="calf_iyz" value="8.28E-06"/>
     <xacro:property name="calf_izz" value="3.29E-05"/>
-    <xacro:property name="foot_mass" value="0.02"/>
+    <!-- foot -->
+    <xacro:property name="foot_mass" value="0.154"/>
 </robot>

File: install/go2_description/share/go2_description/xacro/leg.xacro (robot description, xacro)
@@ -1,4 +1,5 @@
 <?xml version="1.0"?>
 <robot xmlns:xacro="http://www.ros.org/wiki/xacro">
+    <xacro:property name="scale_model" value="2.0"/>
     <!-- <xacro:include filename="$(find go2_description)/xacro/transmission.xacro"/> -->
     <xacro:macro name="leg" params="name mirror mirror_dae front_hind front_hind_dae">
@@ -42,5 +43,5 @@
                 </xacro:if>
                 <geometry>
-                    <mesh filename="file://$(find go2_description)/meshes/${name}_hip_link.STL" scale="1 1 1"/>
+                    <mesh filename="file://$(find go2_description)/meshes/${name}_hip_link.STL" scale="${scale_model} ${scale_model} ${scale_model}"/>
                 </geometry>
                 <!-- <material name="orange"/> -->
@@ -73,5 +74,5 @@
                 <origin rpy="0 0 0" xyz="0 0 0"/>
                 <geometry>
-                    <mesh filename="file://$(find go2_description)/meshes/${name}_upper_leg_link.STL" scale="1 1 1"/>
+                    <mesh filename="file://$(find go2_description)/meshes/${name}_upper_leg_link.STL" scale="${scale_model} ${scale_model} ${scale_model}"/>
                 </geometry>
                 <!-- <material name="orange"/> -->
@@ -104,10 +105,10 @@
                 <origin rpy="0 0 0" xyz="0 0 0"/>
                 <geometry>
-                    <mesh filename="file://$(find go2_description)/meshes/${name}_lower_leg_link.STL" scale="1 1 1"/>
+                    <mesh filename="file://$(find go2_description)/meshes/${name}_lower_leg_link.STL" scale="${scale_model} ${scale_model} ${scale_model}"/>
                 </geometry>
                 <!-- <material name="orange"/> -->
             </visual>
             <collision>
-                <origin rpy="0 ${PI/2.0} 0" xyz="-0.02 ${hip_offset*mirror} -0.03"/>
+                <origin rpy="0 ${PI/2.0} 0" xyz="-0.025 ${hip_offset*mirror} -0.03"/>
                 <geometry>
                     <box size="${calf_length} ${calf_width} ${calf_height}"/>
@@ -130,5 +131,5 @@
         <link name="${name}_foot_link">
             <visual>
-                <origin rpy="0 0 0" xyz="-0.02 ${hip_offset*mirror} -0.03"/>
+                <origin rpy="0 0 0" xyz="-0.05 ${hip_offset*mirror} -0.028"/>
                 <geometry>
                     <sphere radius="${foot_radius-0.01}"/>
@@ -137,13 +138,13 @@
             </visual>
             <collision>
-                <origin rpy="0 0 0" xyz="-0.02 ${hip_offset*mirror} -0.03"/>
+                <origin rpy="0 0 0" xyz="-0.05 ${hip_offset*mirror} -0.028"/>
                 <geometry>
-                    <sphere radius="${foot_radius}"/>
+                    <sphere radius="${foot_radius+0.05}"/>
                 </geometry>
                 <surface>
                     <friction>
                         <ode>
-                            <mu>1.2</mu>
-                            <mu2>1.2</mu2>
+                            <mu>000.2</mu>
+                            <mu2>000.2</mu2>
                         </ode>
                     </friction>

File: install/go2_description/share/go2_description/xacro/robot.xacro (robot description, xacro)
@@ -1,4 +1,4 @@
-<?xml version="1.0"?>
 <robot name="go2" xmlns:xacro="http://www.ros.org/wiki/xacro">
+    <xacro:property name="scale_model" value="2.0"/>
     <xacro:arg name="DEBUG" default="false"/>
     <xacro:include filename="$(find go2_description)/xacro/const.xacro"/>
@@ -37,5 +37,5 @@
             <origin rpy="0 0 0" xyz="0 0 0"/>
             <geometry>
-                <mesh filename="file://$(find go2_description)/meshes/base_link.STL" scale="1 1 1"/>
+                <mesh filename="file://$(find go2_description)/meshes/base_link.STL" scale="${scale_model} ${scale_model} ${scale_model}"/>
             </geometry>
             <!-- <material name="orange"/> -->
